Commit message: legs

File: src/bud_cat/urdf/model.urdf (robot description, URDF)
Before this commit: robot cherry, 1 links, 0 joints
Links:
- added link leg_BL, mass 0.0; collision box size=0.2 0.5 0.03; visual box size=0.2 0.5 0.03
- added link leg_BR, mass 0.0; collision box size=0.2 0.5 0.03; visual box size=0.2 0.5 0.03
- added link leg_FL, mass 0.0; collision box size=0.2 0.5 0.03; visual box size=0.2 0.5 0.03
- added link leg_FR, mass 0.0; collision box size=0.2 0.5 0.03; visual box size=0.2 0.5 0.03
- added link thigh_BL, mass 0.0; collision box size=0.2 0.5 0.03; visual box size=0.2 0.5 0.03
- added link thigh_BR, mass 0.0; collision box size=0.2 0.5 0.03; visual box size=0.2 0.5 0.03
- added link thigh_FL, mass 0.0; collision box size=0.2 0.5 0.03; visual box size=0.2 0.5 0.03
- added link thigh_FR, mass 0.0; collision box size=0.2 0.5 0.03; visual box size=0.2 0.5 0.03
- link base_link: geometry collision box size=1.5 1.0 0.2; visual box size=1.5 1.0 0.2
Joints:
- added joint leg_BL_joint: type revolute, parent thigh_BL, child leg_BL, origin xyz=0 0 0  rpy=0 0.0 0.0, axis 0.0 0.0 0.0, limit lower=0 upper=180 effort=0.1 velocity=0.1
- added joint leg_BR_joint: type revolute, parent thigh_BR, child leg_BR, origin xyz=0 0 0  rpy=0 0.0 0.0, axis 0.0 0.0 0.0, limit lower=0 upper=180 effort=0.1 velocity=0.1
- added joint leg_FL_joint: type revolute, parent thigh_FL, child leg_FL, origin xyz=0 0 0  rpy=0 0.0 0.0, axis 0.0 0.0 0.0, limit lower=0 upper=180 effort=0.1 velocity=0.1
- added joint leg_FR_joint: type revolute, parent thigh_FR, child leg_FR, origin xyz=0 0 0  rpy=0 0.0 0.0, axis 0.0 0.0 0.0, limit lower=0 upper=180 effort=0.1 velocity=0.1
- added joint thigh_BL_joint: type revolute, parent base_link, child thigh_BL, origin xyz=0 0 0  rpy=3.14 0.0 0.0, axis 0.0 0.0 0.0, limit lower=0 upper=180 effort=0.1 velocity=0.1
- added joint thigh_BR_joint: type revolute, parent base_link, child thigh_BR, origin xyz=0 0 0  rpy=3.14 0.0 0.0, axis 0.0 0.0 0.0, limit lower=0 upper=180 effort=0.1 velocity=0.1
- added joint thigh_FL_joint: type revolute, parent base_link, child thigh_FL, origin xyz=0 0 0  rpy=3.14 0.0 0.0, axis 0.0 0.0 0.0, limit lower=0 upper=180 effort=0.1 velocity=0.1
- added joint thigh_FR_joint: type revolute, parent base_link, child thigh_FR, origin xyz=0 0 0  rpy=3.14 0.0 0.0, axis 0.0 0.0 0.0, limit lower=0 upper=180 effort=0.1 velocity=0.1

File: src/bud_cat/urdf/model.xacro (robot description, xacro)
@@ -2,12 +2,39 @@
 <robot xmlns:xacro="http://www.ros.org/wiki/xacro" name="cherry">
 <xacro:property name="body_width" value="1.0" />
-<xacro:property name="body_len" value="1.2" />
+<xacro:property name="body_len" value="1.5" />
 <xacro:property name="body_thickness" value="0.2" />
+<xacro:property name="thickness" value="0.03" />
 <xacro:property name="leg_len" value="0.5" />
 <xacro:property name="hind_len" value="0.5" />
+<xacro:property name="limb_width" value="0.2" />
+<xacro:property name="front_right_limb_x" value="0.5" />
+<xacro:property name="front_right_limb_y" value="0.55" />
+<xacro:property name="front_right_limb_z" value="0.2" />
+<xacro:property name="front_right_leg_x" value="0.5" />
+<xacro:property name="front_right_leg_y" value="0.65" />
+<xacro:property name="front_right_leg_z" value="0.5" />
+<xacro:property name="back_right_limb_x" value="-0.5" />
+<xacro:property name="back_right_limb_y" value="0.55" />
+<xacro:property name="back_right_limb_z" value="0.2" />
+<xacro:property name="back_right_leg_x" value="-0.5" />
+<xacro:property name="back_right_leg_y" value="0.65" />
+<xacro:property name="back_right_leg_z" value="0.5" />
+<xacro:property name="front_left_limb_x" value="0.5" />
+<xacro:property name="front_left_limb_y" value="-0.55" />
+<xacro:property name="front_left_limb_z" value="0.2" />
+<xacro:property name="front_left_leg_x" value="0.5" />
+<xacro:property name="front_left_leg_y" value="-0.65" />
+<xacro:property name="front_left_leg_z" value="0.5" />
+<xacro:property name="back_left_limb_x" value="-0.5" />
+<xacro:property name="back_left_limb_y" value="-0.55" />
+<xacro:property name="back_left_limb_z" value="0.2" />
+<xacro:property name="back_left_leg_x" value="-0.5" />
+<xacro:property name="back_left_leg_y" value="-0.65" />
+<xacro:property name="back_left_leg_z" value="0.5" />
+<!-- <xacro:property name="pi" value="3.14" /> -->
  <link name="base_link">
     <visual>
         <geometry>
-            <box size="${body_width} ${body_len} ${body_thickness}"/>
+           <box size="${body_len} ${body_width} ${body_thickness}"/>
         </geometry>
         <material name="blue"/>
@@ -15,7 +42,264 @@
     <collision>
         <geometry>
-            <box size="${body_width} ${body_len} ${body_thickness}"/>
-        </geometry>
-    </collision>
-</link>
+            <box size="${body_len} ${body_width}  ${body_thickness}"/>
+        </geometry>
+    </collision>
+</link>
+<!-- front right limb -->
+<link name="thigh_FR">
+    <inertial>
+        <origin xyz="0.0 0.0 0.0" rpy="0.0 0.0 0.0"/>
+        <mass value="0.0"/>
+        <inertia ixx="0.0" ixy="0.0" ixz="0.0" iyy="0.0" iyz="0.0" izz="0.0"/>
+    </inertial>
+    <visual name="">
+        <origin xyz="${front_right_limb_x} ${front_right_limb_y} ${front_right_limb_z}" rpy="${pi/2} 0 ${pi/6}"/>
+        <geometry>
+            <box size="${limb_width} ${leg_len} ${thickness} "/>
+        </geometry>
+        <material name="">
+            <color rgba="1.0 0.0 0.0 1.0"/>
+            <texture filename=""/>
+            <texture filename=""/>
+        </material>
+    </visual>
+    <collision>
+        <origin xyz="0.0 0.0 0.0" rpy="0.0 0.0 0.0"/>
+        <geometry>
+            <box size="${limb_width} ${leg_len} ${thickness} "/>
+        </geometry>
+    </collision>
+</link>
+<link name="leg_FR">
+    <inertial>
+        <origin xyz="0.0 0.0 0.0" rpy="0.0 0.0 0.0"/>
+        <mass value="0.0"/>
+        <inertia ixx="0.0" ixy="0.0" ixz="0.0" iyy="0.0" iyz="0.0" izz="0.0"/>
+    </inertial>
+    <visual name="">
+        <origin xyz="${front_right_leg_x} ${front_right_leg_y} ${front_right_leg_z}" rpy="${pi/2} 0 ${-pi/6}"/>
+        <geometry>
+            <box size="${limb_width} ${leg_len} ${thickness} "/>
+        </geometry>
+        <material name="">
+            <color rgba="1.0 0.0 1.0 1.0"/>
+            <texture filename=""/>
+            <texture filename=""/>
+        </material>
+    </visual>
+    <collision>
+        <origin xyz="0.0 0.0 0.0" rpy="0.0 0.0 0.0"/>
+        <geometry>
+            <box size="${limb_width} ${leg_len} ${thickness} "/>
+        </geometry>
+    </collision>
+</link>
+<!-- back right limb -->
+<link name="thigh_BR">
+    <inertial>
+        <origin xyz="0.0 0.0 0.0" rpy="0.0 0.0 0.0"/>
+        <mass value="0.0"/>
+        <inertia ixx="0.0" ixy="0.0" ixz="0.0" iyy="0.0" iyz="0.0" izz="0.0"/>
+    </inertial>
+    <visual name="">
+        <origin xyz="${back_right_limb_x} ${back_right_limb_y} ${back_right_limb_z}" rpy="${pi/2} 0 ${pi/6}"/>
+        <geometry>
+            <box size="${limb_width} ${leg_len} ${thickness} "/>
+        </geometry>
+        <material name="">
+            <color rgba="1.0 0.0 0.0 1.0"/>
+            <texture filename=""/>
+            <texture filename=""/>
+        </material>
+    </visual>
+    <collision>
+        <origin xyz="0.0 0.0 0.0" rpy="0.0 0.0 0.0"/>
+        <geometry>
+            <box size="${limb_width} ${leg_len} ${thickness} "/>
+        </geometry>
+    </collision>
+</link>
+<link name="leg_BR">
+    <inertial>
+        <origin xyz="0.0 0.0 0.0" rpy="0.0 0.0 0.0"/>
+        <mass value="0.0"/>
+        <inertia ixx="0.0" ixy="0.0" ixz="0.0" iyy="0.0" iyz="0.0" izz="0.0"/>
+    </inertial>
+    <visual name="">
+        <origin xyz="${back_right_leg_x} ${back_right_leg_y} ${back_right_leg_z}" rpy="${pi/2} 0 ${-pi/6}"/>
+        <geometry>
+            <box size="${limb_width} ${leg_len} ${thickness} "/>
+        </geometry>
+        <material name="">
+            <color rgba="1.0 0.0 1.0 1.0"/>
+            <texture filename=""/>
+            <texture filename=""/>
+        </material>
+    </visual>
+    <collision>
+        <origin xyz="0.0 0.0 0.0" rpy="0.0 0.0 0.0"/>
+        <geometry>
+            <box size="${limb_width} ${leg_len} ${thickness} "/>
+        </geometry>
+    </collision>
+</link>
+<!-- front right limb -->
+<link name="thigh_FL">
+    <inertial>
+        <origin xyz="0.0 0.0 0.0" rpy="0.0 0.0 0.0"/>
+        <mass value="0.0"/>
+        <inertia ixx="0.0" ixy="0.0" ixz="0.0" iyy="0.0" iyz="0.0" izz="0.0"/>
+    </inertial>
+    <visual name="">
+        <origin xyz="${front_left_limb_x} ${front_left_limb_y} ${front_left_limb_z}" rpy="${pi/2} 0 ${pi/6}"/>
+        <geometry>
+            <box size="${limb_width} ${leg_len} ${thickness} "/>
+        </geometry>
+        <material name="">
+            <color rgba="1.0 0.0 0.0 1.0"/>
+            <texture filename=""/>
+            <texture filename=""/>
+        </material>
+    </visual>
+    <collision>
+        <origin xyz="0.0 0.0 0.0" rpy="0.0 0.0 0.0"/>
+        <geometry>
+            <box size="${limb_width} ${leg_len} ${thickness} "/>
+        </geometry>
+    </collision>
+</link>
+<link name="leg_FL">
+    <inertial>
+        <origin xyz="0.0 0.0 0.0" rpy="0.0 0.0 0.0"/>
+        <mass value="0.0"/>
+        <inertia ixx="0.0" ixy="0.0" ixz="0.0" iyy="0.0" iyz="0.0" izz="0.0"/>
+    </inertial>
+    <visual name="">
+        <origin xyz="${front_left_leg_x} ${front_left_leg_y} ${front_left_leg_z}" rpy="${pi/2} 0 ${-pi/6}"/>
+        <geometry>
+            <box size="${limb_width} ${leg_len} ${thickness} "/>
+        </geometry>
+        <material name="">
+            <color rgba="1.0 0.0 1.0 1.0"/>
+            <texture filename=""/>
+            <texture filename=""/>
+        </material>
+    </visual>
+    <collision>
+        <origin xyz="0.0 0.0 0.0" rpy="0.0 0.0 0.0"/>
+        <geometry>
+            <box size="${limb_width} ${leg_len} ${thickness} "/>
+        </geometry>
+    </collision>
+</link>
+<!-- back right limb -->
+<link name="thigh_BL">
+    <inertial>
+        <origin xyz="0.0 0.0 0.0" rpy="0.0 0.0 0.0"/>
+        <mass value="0.0"/>
+        <inertia ixx="0.0" ixy="0.0" ixz="0.0" iyy="0.0" iyz="0.0" izz="0.0"/>
+    </inertial>
+    <visual name="">
+        <origin xyz="${back_left_limb_x} ${back_left_limb_y} ${back_left_limb_z}" rpy="${pi/2} 0 ${pi/6}"/>
+        <geometry>
+            <box size="${limb_width} ${leg_len} ${thickness} "/>
+        </geometry>
+        <material name="">
+            <color rgba="1.0 0.0 0.0 1.0"/>
+            <texture filename=""/>
+            <texture filename=""/>
+        </material>
+    </visual>
+    <collision>
+        <origin xyz="0.0 0.0 0.0" rpy="0.0 0.0 0.0"/>
+        <geometry>
+            <box size="${limb_width} ${leg_len} ${thickness} "/>
+        </geometry>
+    </collision>
+</link>
+<link name="leg_BL">
+    <inertial>
+        <origin xyz="0.0 0.0 0.0" rpy="0.0 0.0 0.0"/>
+        <mass value="0.0"/>
+        <inertia ixx="0.0" ixy="0.0" ixz="0.0" iyy="0.0" iyz="0.0" izz="0.0"/>
+    </inertial>
+    <visual name="">
+        <origin xyz="${back_left_leg_x} ${back_left_leg_y} ${back_left_leg_z}" rpy="${pi/2} 0 ${-pi/6}"/>
+        <geometry>
+            <box size="${limb_width} ${leg_len} ${thickness} "/>
+        </geometry>
+        <material name="">
+            <color rgba="1.0 0.0 1.0 1.0"/>
+            <texture filename=""/>
+            <texture filename=""/>
+        </material>
+    </visual>
+    <collision>
+        <origin xyz="0.0 0.0 0.0" rpy="0.0 0.0 0.0"/>
+        <geometry>
+            <box size="${limb_width} ${leg_len} ${thickness} "/>
+        </geometry>
+    </collision>
+</link>
+<!-- joints  -->
+<!-- front right limb -->
+<joint name="thigh_FR_joint" type="revolute">
+    <origin xyz="0 0 0 " rpy="3.14 0.0 0.0"/>
+    <parent link="base_link"/>
+    <child link="thigh_FR"/>
+    <axis xyz="0.0 0.0 0.0"/>
+    <limit lower="0" upper="180" effort="0.1" velocity="0.1"/>
+</joint>
+<joint name="leg_FR_joint" type="revolute">
+    <origin xyz="0 0 0 " rpy="0 0.0 0.0"/>
+    <parent link="thigh_FR"/>
+    <child link="leg_FR"/>
+    <axis xyz="0.0 0.0 0.0"/>
+    <limit lower="0" upper="180" effort="0.1" velocity="0.1"/>
+</joint>
+<!-- back right limb -->
+<joint name="thigh_BR_joint" type="revolute">
+    <origin xyz="0 0 0 " rpy="3.14 0.0 0.0"/>
+    <parent link="base_link"/>
+    <child link="thigh_BR"/>
+    <axis xyz="0.0 0.0 0.0"/>
+    <limit lower="0" upper="180" effort="0.1" velocity="0.1"/>
+</joint>
+<joint name="leg_BR_joint" type="revolute">
+    <origin xyz="0 0 0 " rpy="0 0.0 0.0"/>
+    <parent link="thigh_BR"/>
+    <child link="leg_BR"/>
+    <axis xyz="0.0 0.0 0.0"/>
+    <limit lower="0" upper="180" effort="0.1" velocity="0.1"/>
+</joint>
+<!-- front left limb -->
+<joint name="thigh_FL_joint" type="revolute">
+    <origin xyz="0 0 0 " rpy="3.14 0.0 0.0"/>
+    <parent link="base_link"/>
+    <child link="thigh_FL"/>
+    <axis xyz="0.0 0.0 0.0"/>
+    <limit lower="0" upper="180" effort="0.1" velocity="0.1"/>
+</joint>
+<joint name="leg_FL_joint" type="revolute">
+    <origin xyz="0 0 0 " rpy="0 0.0 0.0"/>
+    <parent link="thigh_FL"/>
+    <child link="leg_FL"/>
+    <axis xyz="0.0 0.0 0.0"/>
+    <limit lower="0" upper="180" effort="0.1" velocity="0.1"/>
+</joint>
+<!-- back left limb -->
+<joint name="thigh_BL_joint" type="revolute">
+    <origin xyz="0 0 0 " rpy="3.14 0.0 0.0"/>
+    <parent link="base_link"/>
+    <child link="thigh_BL"/>
+    <axis xyz="0.0 0.0 0.0"/>
+    <limit lower="0" upper="180" effort="0.1" velocity="0.1"/>
+</joint>
+<joint name="leg_BL_joint" type="revolute">
+    <origin xyz="0 0 0 " rpy="0 0.0 0.0"/>
+    <parent link="thigh_BL"/>
+    <child link="leg_BL"/>
+    <axis xyz="0.0 0.0 0.0"/>
+    <limit lower="0" upper="180" effort="0.1" velocity="0.1"/>
+</joint>
 </robot>
