Commit message: urdf

File: src/bud_cat/urdf/model.urdf (robot description, URDF)
Before this commit: robot cherry, 9 links, 8 joints
Links:
- link leg_BL: geometry collision box size=0.1 0.5 0.03; visual box size=0.1 0.5 0.03
- link leg_BR: geometry collision box size=0.1 0.5 0.03; visual box size=0.1 0.5 0.03
- link leg_FL: geometry collision box size=0.1 0.5 0.03; visual box size=0.1 0.5 0.03
- link leg_FR: geometry collision box size=0.1 0.5 0.03; visual box size=0.1 0.5 0.03
- link thigh_BL: geometry collision box size=0.1 0.5 0.03; visual box size=0.1 0.5 0.03
- link thigh_BR: geometry collision box size=0.1 0.5 0.03; visual box size=0.1 0.5 0.03
- link thigh_FL: geometry collision box size=0.1 0.5 0.03; visual box size=0.1 0.5 0.03
- link thigh_FR: geometry collision box size=0.1 0.5 0.03; visual box size=0.1 0.5 0.03
Joints:
- joint leg_BL_joint: axis 0.0 0.0 0.0 -> 0.0 1.0 0.0; limit lower=0 upper=180 effort=0.1 velocity=0.1 -> lower=-1.5707963267948966 upper=1.5707963267948966 effort=0.1 velocity=10; origin xyz=0 0 0  rpy=0 0.0 0.0 -> xyz=0 0 -0.4 rpy=0 0.0 0.0
- joint leg_BR_joint: axis 0.0 0.0 0.0 -> 0.0 1.0 0.0; limit lower=0 upper=180 effort=0.1 velocity=0.1 -> lower=-1.5707963267948966 upper=1.5707963267948966 effort=0.1 velocity=10; origin xyz=0 0 0  rpy=0 0.0 0.0 -> xyz=0 0 -0.4 rpy=0 0.0 0.0
- joint leg_FL_joint: axis 0.0 0.0 0.0 -> 0.0 1.0 0.0; limit lower=0 upper=180 effort=0.1 velocity=0.1 -> lower=-1.5707963267948966 upper=1.5707963267948966 effort=0.1 velocity=10; origin xyz=0 0 0  rpy=0 0.0 0.0 -> xyz=0 0 -0.4 rpy=0 0.0 0.0
- joint leg_FR_joint: axis 0.0 0.0 0.0 -> 0.0 1.0 0.0; limit lower=0 upper=180 effort=0.1 velocity=0.1 -> lower=-1.5707963267948966 upper=1.5707963267948966 effort=0.1 velocity=10; origin xyz=0 0 0  rpy=0 0.0 0.0 -> xyz=0 0 -0.4 rpy=0 0.0 0.0
- joint thigh_BL_joint: axis 0.0 0.0 0.0 -> 0.0 1.0 0.0; limit lower=0 upper=180 effort=0.1 velocity=0.1 -> lower=-1.5707963267948966 upper=1.5707963267948966 effort=0.1 velocity=10; origin xyz=0 0 0  rpy=3.14 0.0 0.0 -> xyz=-0.5 -0.5 0 rpy=0 0.0 0.0
- joint thigh_BR_joint: axis 0.0 0.0 0.0 -> 0.0 1.0 0.0; limit lower=0 upper=180 effort=0.1 velocity=0.1 -> lower=-1.5707963267948966 upper=1.5707963267948966 effort=0.1 velocity=10; origin xyz=0 0 0  rpy=3.14 0.0 0.0 -> xyz=-0.5 0.5 0 rpy=0 0.0 0.0
- joint thigh_FL_joint: axis 0.0 0.0 0.0 -> 0.0 1.0 0.0; limit lower=0 upper=180 effort=0.1 velocity=0.1 -> lower=-1.5707963267948966 upper=1.5707963267948966 effort=0.1 velocity=10; origin xyz=0 0 0  rpy=3.14 0.0 0.0 -> xyz=0.5 -0.5 0 rpy=0 0.0 0.0
- joint thigh_FR_joint: axis 0.0 0.0 0.0 -> 0.0 1.0 0.0; limit lower=0 upper=180 effort=0.1 velocity=0.1 -> lower=-1.5707963267948966 upper=1.5707963267948966 effort=0.1 velocity=10; origin xyz=0 0 0  rpy=3.14 0.0 0.0 -> xyz=0.5 0.5 0 rpy=0 0.0 0.0

File: src/bud_cat/urdf/model_bck.xacro (robot description, xacro)
@@ -7,34 +7,30 @@
 <xacro:property name="leg_len" value="0.5" />
 <xacro:property name="hind_len" value="0.5" />
-<xacro:property name="limb_width" value="0.1" />
-<xacro:property name="joint_vel" value="10" />
+<xacro:property name="limb_width" value="0.2" />
 <xacro:property name="front_right_limb_x" value="0.5" />
-<xacro:property name="front_right_limb_y" value="0.5" />
-<xacro:property name="front_right_limb_z" value="-0.2" />
-<xacro:property name="front_right_leg_x" value="0" />
-<xacro:property name="front_right_leg_y" value="0" />
-<xacro:property name="front_right_leg_z" value="-0.4" />
-<xacro:property name="front_right_leg_joint_z" value="-0.2" />
+<xacro:property name="front_right_limb_y" value="0.55" />
+<xacro:property name="front_right_limb_z" value="0.2" />
+<xacro:property name="front_right_leg_x" value="0.5" />
+<xacro:property name="front_right_leg_y" value="0.65" />
+<xacro:property name="front_right_leg_z" value="0.5" />
 <xacro:property name="back_right_limb_x" value="-0.5" />
-<xacro:property name="back_right_limb_y" value="0.5" />
-<xacro:property name="back_right_limb_z" value="-0.2" />
-<xacro:property name="back_right_leg_x" value="0" />
-<xacro:property name="back_right_leg_y" value="0" />
-<xacro:property name="back_right_leg_z" value="-0.4" />
-<xacro:property name="back_right_leg_joint_z" value="-0.2" />
+<xacro:property name="back_right_limb_y" value="0.55" />
+<xacro:property name="back_right_limb_z" value="0.2" />
+<xacro:property name="back_right_leg_x" value="-0.5" />
+<xacro:property name="back_right_leg_y" value="0.65" />
+<xacro:property name="back_right_leg_z" value="0.5" />
 <xacro:property name="front_left_limb_x" value="0.5" />
-<xacro:property name="front_left_limb_y" value="-0.5" />
-<xacro:property name="front_left_limb_z" value="-0.2" />
-<xacro:property name="front_left_leg_x" value="0" />
-<xacro:property name="front_left_leg_y" value="0" />
-<xacro:property name="front_left_leg_z" value="-0.4" />
-<xacro:property name="front_left_leg_joint_z" value="-0.2" />
+<xacro:property name="front_left_limb_y" value="-0.55" />
+<xacro:property name="front_left_limb_z" value="0.2" />
+<xacro:property name="front_left_leg_x" value="0.5" />
+<xacro:property name="front_left_leg_y" value="-0.65" />
+<xacro:property name="front_left_leg_z" value="0.5" />
 <xacro:property name="back_left_limb_x" value="-0.5" />
-<xacro:property name="back_left_limb_y" value="-0.5" />
-<xacro:property name="back_left_limb_z" value="-0.2" />
-<xacro:property name="back_left_leg_x" value="0" />
-<xacro:property name="back_left_leg_y" value="0" />
-<xacro:property name="back_left_leg_z" value="-0.4" />
-<xacro:property name="back_left_leg_joint_z" value="-0.2" />
+<xacro:property name="back_left_limb_y" value="-0.55" />
+<xacro:property name="back_left_limb_z" value="0.2" />
+<xacro:property name="back_left_leg_x" value="-0.5" />
+<xacro:property name="back_left_leg_y" value="-0.65" />
+<xacro:property name="back_left_leg_z" value="0.5" />
+<!-- <xacro:property name="pi" value="3.14" /> -->
  <link name="base_link">
     <visual>
@@ -49,28 +45,14 @@
         </geometry>
     </collision>
-    <inertial>
-        <origin xyz="0.0 0.0 0.0" rpy="0.0 0.0 0.0"/>
-        <mass value="0.5"/>
-        <geometry>
-            <box size="${body_len} ${body_width}  ${body_thickness}"/>
-        </geometry>
-    </inertial>
-    <collision>
-        <geometry>
-            <box size="${body_len} ${body_width}  ${body_thickness}"/>
-        </geometry>
-    </collision>
 </link>
 <!-- front right limb -->
 <link name="thigh_FR">
     <inertial>
-        <origin xyz="0 0 ${front_right_limb_z}" rpy="${pi/2} 0 0 "/>
-        <mass value="0.1"/>
-        <geometry>
-            <box size="${body_len} ${body_width}  ${body_thickness}"/>
-        </geometry>
-    </inertial>
-    <visual name="">
-        <origin xyz="0 0 ${front_right_limb_z}" rpy="${pi/2} 0 0 "/>
+        <origin xyz="0.0 0.0 0.0" rpy="0.0 0.0 0.0"/>
+        <mass value="0.0"/>
+        <inertia ixx="0.0" ixy="0.0" ixz="0.0" iyy="0.0" iyz="0.0" izz="0.0"/>
+    </inertial>
+    <visual name="">
+        <origin xyz="${front_right_limb_x} ${front_right_limb_y} ${front_right_limb_z}" rpy="${pi/2} 0 ${pi/6}"/>
         <geometry>
             <box size="${limb_width} ${leg_len} ${thickness} "/>
@@ -96,5 +78,5 @@
     </inertial>
     <visual name="">
-        <origin xyz="0 0 ${front_right_leg_joint_z}" rpy="${pi/2} 0 0"/>
+        <origin xyz="${front_right_leg_x} ${front_right_leg_y} ${front_right_leg_z}" rpy="${pi/2} 0 ${-pi/6}"/>
         <geometry>
             <box size="${limb_width} ${leg_len} ${thickness} "/>
@@ -113,13 +95,62 @@
     </collision>
 </link>
+<!-- back right limb -->
+<link name="thigh_BR">
+    <inertial>
+        <origin xyz="0.0 0.0 0.0" rpy="0.0 0.0 0.0"/>
+        <mass value="0.0"/>
+        <inertia ixx="0.0" ixy="0.0" ixz="0.0" iyy="0.0" iyz="0.0" izz="0.0"/>
+    </inertial>
+    <visual name="">
+        <origin xyz="${back_right_limb_x} ${back_right_limb_y} ${back_right_limb_z}" rpy="${pi/2} 0 ${pi/6}"/>
+        <geometry>
+            <box size="${limb_width} ${leg_len} ${thickness} "/>
+        </geometry>
+        <material name="">
+            <color rgba="1.0 0.0 0.0 1.0"/>
+            <texture filename=""/>
+            <texture filename=""/>
+        </material>
+    </visual>
+    <collision>
+        <origin xyz="0.0 0.0 0.0" rpy="0.0 0.0 0.0"/>
+        <geometry>
+            <box size="${limb_width} ${leg_len} ${thickness} "/>
+        </geometry>
+    </collision>
+</link>
+<link name="leg_BR">
+    <inertial>
+        <origin xyz="0.0 0.0 0.0" rpy="0.0 0.0 0.0"/>
+        <mass value="0.0"/>
+        <inertia ixx="0.0" ixy="0.0" ixz="0.0" iyy="0.0" iyz="0.0" izz="0.0"/>
+    </inertial>
+    <visual name="">
+        <origin xyz="${back_right_leg_x} ${back_right_leg_y} ${back_right_leg_z}" rpy="${pi/2} 0 ${-pi/6}"/>
+        <geometry>
+            <box size="${limb_width} ${leg_len} ${thickness} "/>
+        </geometry>
+        <material name="">
+            <color rgba="1.0 0.0 1.0 1.0"/>
+            <texture filename=""/>
+            <texture filename=""/>
+        </material>
+    </visual>
+    <collision>
+        <origin xyz="0.0 0.0 0.0" rpy="0.0 0.0 0.0"/>
+        <geometry>
+            <box size="${limb_width} ${leg_len} ${thickness} "/>
+        </geometry>
+    </collision>
+</link>
 <!-- front right limb -->
-<link name="thigh_BR">
-    <inertial>
-        <origin xyz="0.0 0.0 0.0" rpy="0.0 0.0 0.0"/>
-        <mass value="0.0"/>
-        <inertia ixx="0.0" ixy="0.0" ixz="0.0" iyy="0.0" iyz="0.0" izz="0.0"/>
-    </inertial>
-    <visual name="">
-        <origin xyz="0 0 ${back_right_limb_z}" rpy="${pi/2} 0 0 "/>
+<link name="thigh_FL">
+    <inertial>
+        <origin xyz="0.0 0.0 0.0" rpy="0.0 0.0 0.0"/>
+        <mass value="0.0"/>
+        <inertia ixx="0.0" ixy="0.0" ixz="0.0" iyy="0.0" iyz="0.0" izz="0.0"/>
+    </inertial>
+    <visual name="">
+        <origin xyz="${front_left_limb_x} ${front_left_limb_y} ${front_left_limb_z}" rpy="${pi/2} 0 ${pi/6}"/>
         <geometry>
             <box size="${limb_width} ${leg_len} ${thickness} "/>
@@ -138,12 +169,12 @@
     </collision>
 </link>
-<link name="leg_BR">
-    <inertial>
-        <origin xyz="0.0 0.0 0.0" rpy="0.0 0.0 0.0"/>
-        <mass value="0.0"/>
-        <inertia ixx="0.0" ixy="0.0" ixz="0.0" iyy="0.0" iyz="0.0" izz="0.0"/>
-    </inertial>
-    <visual name="">
-        <origin xyz="0 0 ${back_right_leg_joint_z}" rpy="${pi/2} 0 0"/>
+<link name="leg_FL">
+    <inertial>
+        <origin xyz="0.0 0.0 0.0" rpy="0.0 0.0 0.0"/>
+        <mass value="0.0"/>
+        <inertia ixx="0.0" ixy="0.0" ixz="0.0" iyy="0.0" iyz="0.0" izz="0.0"/>
+    </inertial>
+    <visual name="">
+        <origin xyz="${front_left_leg_x} ${front_left_leg_y} ${front_left_leg_z}" rpy="${pi/2} 0 ${-pi/6}"/>
         <geometry>
             <box size="${limb_width} ${leg_len} ${thickness} "/>
@@ -162,13 +193,13 @@
     </collision>
 </link>
-<!-- front left limb -->
-<link name="thigh_FL">
-    <inertial>
-        <origin xyz="0.0 0.0 0.0" rpy="0.0 0.0 0.0"/>
-        <mass value="0.0"/>
-        <inertia ixx="0.0" ixy="0.0" ixz="0.0" iyy="0.0" iyz="0.0" izz="0.0"/>
-    </inertial>
-    <visual name="">
-        <origin xyz="0 0 ${front_left_limb_z}" rpy="${pi/2} 0 0 "/>
+<!-- back right limb -->
+<link name="thigh_BL">
+    <inertial>
+        <origin xyz="0.0 0.0 0.0" rpy="0.0 0.0 0.0"/>
+        <mass value="0.0"/>
+        <inertia ixx="0.0" ixy="0.0" ixz="0.0" iyy="0.0" iyz="0.0" izz="0.0"/>
+    </inertial>
+    <visual name="">
+        <origin xyz="${back_left_limb_x} ${back_left_limb_y} ${back_left_limb_z}" rpy="${pi/2} 0 ${pi/6}"/>
         <geometry>
             <box size="${limb_width} ${leg_len} ${thickness} "/>
@@ -187,53 +218,4 @@
     </collision>
 </link>
-<link name="leg_FL">
-    <inertial>
-        <origin xyz="0.0 0.0 0.0" rpy="0.0 0.0 0.0"/>
-        <mass value="0.0"/>
-        <inertia ixx="0.0" ixy="0.0" ixz="0.0" iyy="0.0" iyz="0.0" izz="0.0"/>
-    </inertial>
-    <visual name="">
-        <origin xyz="0 0 ${front_left_leg_joint_z}" rpy="${pi/2} 0 0"/>
-        <geometry>
-            <box size="${limb_width} ${leg_len} ${thickness} "/>
-        </geometry>
-        <material name="">
-            <color rgba="1.0 0.0 1.0 1.0"/>
-            <texture filename=""/>
-            <texture filename=""/>
-        </material>
-    </visual>
-    <collision>
-        <origin xyz="0.0 0.0 0.0" rpy="0.0 0.0 0.0"/>
-        <geometry>
-            <box size="${limb_width} ${leg_len} ${thickness} "/>
-        </geometry>
-    </collision>
-</link>
-<!-- back left limb -->
-<link name="thigh_BL">
-    <inertial>
-        <origin xyz="0.0 0.0 0.0" rpy="0.0 0.0 0.0"/>
-        <mass value="0.0"/>
-        <inertia ixx="0.0" ixy="0.0" ixz="0.0" iyy="0.0" iyz="0.0" izz="0.0"/>
-    </inertial>
-    <visual name="">
-        <origin xyz="0 0 ${back_left_limb_z}" rpy="${pi/2} 0 0 "/>
-        <geometry>
-            <box size="${limb_width} ${leg_len} ${thickness} "/>
-        </geometry>
-        <material name="">
-            <color rgba="1.0 0.0 0.0 1.0"/>
-            <texture filename=""/>
-            <texture filename=""/>
-        </material>
-    </visual>
-    <collision>
-        <origin xyz="0.0 0.0 0.0" rpy="0.0 0.0 0.0"/>
-        <geometry>
-            <box size="${limb_width} ${leg_len} ${thickness} "/>
-        </geometry>
-    </collision>
-</link>
 <link name="leg_BL">
     <inertial>
@@ -243,5 +225,5 @@
     </inertial>
     <visual name="">
-        <origin xyz="0 0 ${back_left_leg_joint_z}" rpy="${pi/2} 0 0"/>
+        <origin xyz="${back_left_leg_x} ${back_left_leg_y} ${back_left_leg_z}" rpy="${pi/2} 0 ${-pi/6}"/>
         <geometry>
             <box size="${limb_width} ${leg_len} ${thickness} "/>
@@ -263,24 +245,24 @@
 <!-- front right limb -->
 <joint name="thigh_FR_joint" type="revolute">
-    <origin xyz="${front_right_limb_x} ${front_right_limb_y} 0" rpy="0 0.0 0.0"/>
+    <origin xyz="${front_right_limb_x} ${front_right_limb_y} ${front_right_limb_z}" rpy="3.14 0.0 0.0"/>
     <parent link="base_link"/>
     <child link="thigh_FR"/>
-    <axis xyz="0.0 1.0 0.0"/>
-    <limit lower="-${pi/2}" upper="${pi/2}" effort="0.1" velocity="${joint_vel}"/>
+    <axis xyz="0.0 0.0 0.0"/>
+    <limit lower="0" upper="180" effort="0.1" velocity="0.1"/>
 </joint>
 <joint name="leg_FR_joint" type="revolute">
-    <origin xyz="${front_right_leg_x} ${front_right_leg_y} ${front_right_leg_z}" rpy="0 0.0 0.0"/>
+    <origin xyz="${front_right_leg_x} ${front_right_leg_y} ${front_right_leg_z}"  rpy="0 0.0 0.0"/>
     <parent link="thigh_FR"/>
     <child link="leg_FR"/>
-    <axis xyz="0.0 1.0 0.0"/>
-    <limit lower="-${pi/2}" upper="${pi/2}" effort="0.1" velocity="${joint_vel}"/>
+    <axis xyz="0.0 0.0 0.0"/>
+    <limit lower="0" upper="180" effort="0.1" velocity="0.1"/>
 </joint>
 <!-- back right limb -->
 <joint name="thigh_BR_joint" type="revolute">
-    <origin xyz="${back_right_limb_x} ${back_right_limb_y} 0" rpy="0 0.0 0.0"/>
+    <origin xyz="${back_right_limb_x} ${back_right_limb_y} ${back_right_limb_z}" rpy="3.14 0.0 0.0"/>
     <parent link="base_link"/>
     <child link="thigh_BR"/>
-    <axis xyz="0.0 1.0 0.0"/>
-    <limit lower="-${pi/2}" upper="${pi/2}" effort="0.1" velocity="${joint_vel}"/>
+    <axis xyz="0.0 0.0 0.0"/>
+    <limit lower="0" upper="180" effort="0.1" velocity="0.1"/>
 </joint>
 <joint name="leg_BR_joint" type="revolute">
@@ -288,36 +270,36 @@
     <parent link="thigh_BR"/>
     <child link="leg_BR"/>
-    <axis xyz="0.0 1.0 0.0"/>
-    <limit lower="-${pi/2}" upper="${pi/2}" effort="0.1" velocity="${joint_vel}"/>
+    <axis xyz="0.0 0.0 0.0"/>
+    <limit lower="0" upper="180" effort="0.1" velocity="0.1"/>
 </joint>
 <!-- front left limb -->
 <joint name="thigh_FL_joint" type="revolute">
-    <origin xyz="${front_left_limb_x} ${front_left_limb_y} 0" rpy="0 0.0 0.0"/>
+    <origin xyz="${front_left_limb_x} ${front_left_limb_y} ${front_left_limb_z}" rpy="3.14 0.0 0.0"/>
     <parent link="base_link"/>
     <child link="thigh_FL"/>
-    <axis xyz="0.0 1.0 0.0"/>
-    <limit lower="-${pi/2}" upper="${pi/2}" effort="0.1" velocity="${joint_vel}"/>
+    <axis xyz="0.0 0.0 0.0"/>
+    <limit lower="0" upper="180" effort="0.1" velocity="0.1"/>
 </joint>
 <joint name="leg_FL_joint" type="revolute">
-    <origin xyz="${front_left_leg_x} ${front_left_leg_y} ${front_left_leg_z}" rpy="0 0.0 0.0"/>
+    <origin xyz="${front_left_leg_x} ${front_left_leg_y} ${front_left_leg_z} " rpy="0 0.0 0.0"/>
     <parent link="thigh_FL"/>
     <child link="leg_FL"/>
-    <axis xyz="0.0 1.0 0.0"/>
-    <limit lower="-${pi/2}" upper="${pi/2}" effort="0.1" velocity="${joint_vel}"/>
+    <axis xyz="0.0 0.0 0.0"/>
+    <limit lower="0" upper="180" effort="0.1" velocity="0.1"/>
 </joint>
 <!-- back left limb -->
 <joint name="thigh_BL_joint" type="revolute">
-    <origin xyz="${back_left_limb_x} ${back_left_limb_y} 0" rpy="0 0.0 0.0"/>
+    <origin xyz="${back_left_limb_x} ${back_left_limb_y} ${back_left_limb_z}" rpy="3.14 0.0 0.0"/>
     <parent link="base_link"/>
     <child link="thigh_BL"/>
-    <axis xyz="0.0 1.0 0.0"/>
-    <limit lower="-${pi/2}" upper="${pi/2}" effort="0.1" velocity="${joint_vel}"/>
+    <axis xyz="0.0 0.0 0.0"/>
+    <limit lower="0" upper="180" effort="0.1" velocity="0.1"/>
 </joint>
 <joint name="leg_BL_joint" type="revolute">
-    <origin xyz="${back_left_leg_x} ${back_left_leg_y} ${back_left_leg_z}" rpy="0 0.0 0.0"/>
+    <origin xyz="${back_left_leg_x} ${back_left_leg_y} ${back_left_leg_z}" rpy="0 0 0"/>
     <parent link="thigh_BL"/>
     <child link="leg_BL"/>
-    <axis xyz="0.0 1.0 0.0"/>
-    <limit lower="-${pi/2}" upper="${pi/2}" effort="0.1" velocity="${joint_vel}"/>
+    <axis xyz="0.0 0.0 0.0"/>
+    <limit lower="0" upper="180" effort="0.1" velocity="0.1"/>
 </joint>
 </robot>

Commit message: blabla

File: src/bud_cat/urdf/model.urdf (robot description, URDF)
Before this commit: robot cherry, 9 links, 8 joints
Links:
- link base_link: mass None -> 0.5; geometry collision box size=1.5 1.0 0.2; collision box size=1.5 1.0 0.2
- link thigh_FR: mass 0.0 -> 0.1
